Commit message: Add LiDAR yaw property and update joint origin for lidar_joint

File: src/puzzlebot_description/urdf/puzzlebot_mcr2.urdf.xacro (robot description, xacro)
@@ -14,4 +14,7 @@
   <xacro:property name="wheel_mass" value="0.1"/>
   <xacro:property name="caster_mass" value="0.01"/>
+  <!-- LiDAR mounting yaw — physical RPLidar A1 on the MCR2 ships rotated 180°
+       (motor/cable facing rear); Gazebo's gpu_lidar emits ray 0 along +X. -->
+  <xacro:property name="lidar_yaw" value="${0.0 if '$(arg is_sim)' == 'true' else 3.141592653589793}"/>
   <!-- Inertia macros -->
   <xacro:macro name="cylinder_inertia" params="m r h">
@@ -161,5 +164,5 @@
     <parent link="base_link"/>
     <child link="lidar_link"/>
-    <origin xyz="0.05 0 0.110" rpy="0 0 0"/>
+    <origin xyz="0.05 0 0.110" rpy="0 0 ${lidar_yaw}"/>
   </joint>
   <!-- base_link -> camera_link -->
